File: pcb/macropad.kicad_sch (KiCad schematic)
At the start: 15 parts, among them SW1 SW_Push, SW2 SW_Push, SW3 SW_Push, SW4 SW_Push, SW5 SW_Push, SW6 SW_Push, U1 SEEED STUDIO XIAO RP2040, U2 1x0.91 IN. OLED

Commit message: Update images without display
Other:
- title: Physical Control Center -> PCC (Physical Control Center)
Changed lines of the file:
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@@
 	(generator "eeschema")
 	(generator_version "10.0")
-	(paper "A4")
+	(paper "USLetter")
 	(title_block
-		(title "Physical Control Center")
+		(title "PCC (Physical Control Center)")
 		(date "2026-06-10")
-		(rev "1.0")
+		(rev "1.4")
 	)
 	(junction
